Commit message: Add files via upload

File: mybot/urdf/mybot.xacro (robot description, xacro)
@@ -152,3 +152,29 @@
       xyz="0 0 1" />
   </joint>
+  <!--Add transmission for joints of my bot here-->
+  <transmission name="trans_fly_wheel_joint">
+    <type>transmission_interface/SimpleTransmission</type>
+    <joint name="fly_wheel_joint">
+        <hardwareInterface>hardwareInterface/EffortJointInterface</hardwareInterface>
+    </joint>
+    <actuator name="motor_fly_wheel_joint">
+        <hardwareInterface>hardware_interface/EffortJointInterface</hardwareInterface>
+        <mechanicalReduction>1</mechanicalReduction>
+    </actuator>
+  </transmission>
+  <transmission name="trans_wheel_joint">
+    <type>transmission_interface/SimpleTransmission</type>
+    <joint name = "wheel_joint">
+        <hardwareInterface>hardwareInterface/EffortJointInterface</hardwareInterface>
+    </joint>
+    <actuator name="motor_wheel_joint">
+        <hardwareInterface>hardware_interface/EffortJointInterface</hardwareInterface>
+        <mechanicalReduction>1</mechanicalReduction>
+    </actuator>
+  </transmission>
+  <!--Add a gazebo controller plugin here-->
+  <gazebo>
+    <plugin name="gazebo_ros_control" filename="libgazebo_ros_control.so">
+    </plugin>
+  </gazebo>
 </robot>
